File: PDB.kicad_pcb (KiCad board)
At the start: 2 copper layers, 97 x 46 mm, 15 parts, among them J1 Screw_Terminal_01x02, J2 Barrel_Jack_MountingPin, J3 Barrel_Jack_MountingPin, J4 Barrel_Jack_MountingPin, J5 Barrel_Jack_MountingPin, U1 D-SUN(green)_SDC, U2 D-SUN(green)_SDC, U3 D-SUN(green)_SDC, U4 D-SUN(green)_SDC

Commit message: Add files via upload
Parts:
- added J6: Conn_01x04_Female, Connector_JST:JST_PH_B4B-PH-K_1x04_P2.00mm_Vertical, F.Cu at (101.0, 25.0)
- added U5: D-SUN(green)_SDC, Step-down converters:D-SUN(green) SDC, F.Cu at (54.0, 45.0)
- added U6: Wemos-ESP32-S2-Mini, Wemos ESP-32 S2 Mini:Wemos ESP-32 S2 Mini, F.Cu at (77.0, 38.0)
- added U7: EasyDrive, Stepper motor driver:EasyDriver, F.Cu at (118.0, 42.0)
- moved REF** 32.0 mm to (136.0, 25.0)
- moved REF** 32.0 mm to (49.0, 25.0)
Routing:
- net Net-(U6-Pad33): track 0.00 -> 82.6 mm
- net Net-(U6-PadGND_OUTER): track 0.00 -> 75.0 mm, vias 0 -> 1
- net Net-(U6-Pad21): track 0.00 -> 74.9 mm, vias 0 -> 1
- net Net-(U6-Pad18): track 0.00 -> 67.4 mm
- net Net-(U6-Pad5): track 0.00 -> 55.5 mm, vias 0 -> 1
- net Net-(J1-Pad1): track 93.3 -> 145.7 mm
- net Net-(J1-Pad2): track 129.2 -> 176.1 mm
- net Net-(U5-Pad7): track 0.00 -> 32.5 mm
- net Net-(J6-Pad4): track 0.00 -> 9.73 mm
- net Net-(J6-Pad1): track 0.00 -> 9.70 mm
- net Net-(J6-Pad3): track 0.00 -> 9.50 mm
- net Net-(J6-Pad2): track 0.00 -> 9.48 mm
- net Net-(U5-Pad5): track 0.00 -> 8.40 mm
Other:
- board size 97 x 46 mm -> 97 x 78 mm
